File: hardware/ws2812_23sch.sch (KiCad schematic (older format))
At the start: 64 parts

Commit message: update,
Parts:
- removed D? (x40): WS2812B, footprint-lib:LED_WS2812B_PLCC4_5.0x5.0mm_P3.2mm, symbol LED:WS2812B
- added D100, D103, D105, D107, D108, D111, D112, D116, D117, D118, D119, D120, D121, D123, D124, D125, D127, D128, D65, D69, D72, D73, D75, D78, D79, D80, D81, D82, D83, D84, D85, D86, D87, D89, D90, D91, D92, D93, D94, D97: WS2812B, footprint-lib:LED_WS2812B_PLCC4_5.0x5.0mm_P3.2mm, symbol LED:WS2812B
- gave numbers to parts that had none: 24
Connections:
- net GND: now also D100.3 (VSS), D103.3 (VSS), D105.3 (VSS), D107.3 (VSS), D108.3 (VSS), D111.3 (VSS), D112.3 (VSS), D116.3 (VSS), D117.3 (VSS), D118.3 (VSS), D119.3 (VSS), D120.3 (VSS), D121.3 (VSS), D123.3 (VSS), D124.3 (VSS), D125.3 (VSS), D127.3 (VSS), D128.3 (VSS), D65.3 (VSS), D69.3 (VSS), D72.3 (VSS), D73.3 (VSS), D75.3 (VSS), D78.3 (VSS), D79.3 (VSS), D80.3 (VSS), D81.3 (VSS), D82.3 (VSS), D83.3 (VSS), D84.3 (VSS), D85.3 (VSS), D86.3 (VSS), D87.3 (VSS), D89.3 (VSS), D90.3 (VSS), D91.3 (VSS), D92.3 (VSS), D93.3 (VSS), D94.3 (VSS), D97.3 (VSS)
- net VDD: now also D100.1 (VDD), D103.1 (VDD), D105.1 (VDD), D107.1 (VDD), D108.1 (VDD), D111.1 (VDD), D112.1 (VDD), D116.1 (VDD), D117.1 (VDD), D118.1 (VDD), D119.1 (VDD), D120.1 (VDD), D121.1 (VDD), D123.1 (VDD), D124.1 (VDD), D125.1 (VDD), D127.1 (VDD), D128.1 (VDD), D65.1 (VDD), D69.1 (VDD), D72.1 (VDD), D73.1 (VDD), D75.1 (VDD), D78.1 (VDD), D79.1 (VDD), D80.1 (VDD), D81.1 (VDD), D82.1 (VDD), D83.1 (VDD), D84.1 (VDD), D85.1 (VDD), D86.1 (VDD), D87.1 (VDD), D89.1 (VDD), D90.1 (VDD), D91.1 (VDD), D92.1 (VDD), D93.1 (VDD), D94.1 (VDD), D97.1 (VDD)
- net WS2812_IN_ROW1: now also D65.4 (DIN)
- net WS2812_IN_ROW2: now also D73.4 (DIN)
- net WS2812_IN_ROW3: now also D81.4 (DIN)
- net WS2812_IN_ROW4: now also D89.4 (DIN)
- net WS2812_IN_ROW5: now also D97.4 (DIN)
- net WS2812_IN_ROW6: now also D105.4 (DIN)
- net WS2812_IN_ROW8: now also D121.4 (DIN)
- net WS2812_OUT_ROW1: now also D72.2 (DOUT)
- net WS2812_OUT_ROW2: now also D80.2 (DOUT)
- net WS2812_OUT_ROW6: now also D112.2 (DOUT)
- net WS2812_OUT_ROW7: now also D120.2 (DOUT)
- net WS2812_OUT_ROW8: now also D128.2 (DOUT)
- net at D66.4 (DIN): now also D65.2 (DOUT)
- net at D70.4 (DIN): now also D69.2 (DOUT)
- net at D68.2 (DOUT): now also D69.4 (DIN)
- net at D71.2 (DOUT): now also D72.4 (DIN)
- net at D76.4 (DIN): now also D75.2 (DOUT)
- net at D88.4 (DIN): now also D87.2 (DOUT)
- net at D101.4 (DIN): now also D100.2 (DOUT)
- net at D99.2 (DOUT): now also D100.4 (DIN)
- net at D104.4 (DIN): now also D103.2 (DOUT)
- net at D102.2 (DOUT): now also D103.4 (DIN)
- net at D126.4 (DIN): now also D125.2 (DOUT)
- net at D126.2 (DOUT): now also D127.4 (DIN)
- net at D74.4 (DIN): now also D73.2 (DOUT)
- net at D74.2 (DOUT): now also D75.4 (DIN)
- net at D77.2 (DOUT): now also D78.4 (DIN)
- net at D106.4 (DIN): now also D105.2 (DOUT)
- net at D110.2 (DOUT): now also D111.4 (DIN)
- net at D95.4 (DIN): now also D94.2 (DOUT)
- net at D106.2 (DOUT): now also D107.4 (DIN)
- net at D115.2 (DOUT): now also D116.4 (DIN)
- net at D122.4 (DIN): now also D121.2 (DOUT)
- net at D122.2 (DOUT): now also D123.4 (DIN)
- net at D98.4 (DIN): now also D97.2 (DOUT)
- net at D109.4 (DIN): now also D108.2 (DOUT)
- new net: D81.2 (DOUT), D82.4 (DIN)
- new net: D82.2 (DOUT), D83.4 (DIN)
- new net: D85.2 (DOUT), D86.4 (DIN)
- new net: D84.2 (DOUT), D85.4 (DIN)
- new net: D86.2 (DOUT), D87.4 (DIN)
- new net: D119.2 (DOUT), D120.4 (DIN)
- new net: D118.2 (DOUT), D119.4 (DIN)
- new net: D124.2 (DOUT), D125.4 (DIN)
- new net: D123.2 (DOUT), D124.4 (DIN)
- new net: D78.2 (DOUT), D79.4 (DIN)
- new net: D79.2 (DOUT), D80.4 (DIN)
- new net: D89.2 (DOUT), D90.4 (DIN)
- new net: D90.2 (DOUT), D91.4 (DIN)
- new net: D91.2 (DOUT), D92.4 (DIN)
- new net: D92.2 (DOUT), D93.4 (DIN)
- new net: D83.2 (DOUT), D84.4 (DIN)
- new net: D93.2 (DOUT), D94.4 (DIN)
- new net: D111.2 (DOUT), D112.4 (DIN)
- new net: D116.2 (DOUT), D117.4 (DIN)
- new net: D117.2 (DOUT), D118.4 (DIN)
- new net: D127.2 (DOUT), D128.4 (DIN)
- new net: D107.2 (DOUT), D108.4 (DIN)
