File: hardware/follower_counter_tryout.sch (KiCad schematic (older format))
At the start: 0 parts

Commit message: update,
Parts:
- added J?: Conn_01x03, symbol Connector_Generic:Conn_01x03
Connections:
- new net GND: J?.3 (Pin_3)
- new net VDD: J?.1 (Pin_1)
- new net ws2812_01/WS2812_IN_ROW8: J?.2 (Pin_2)
Changed lines of the file:
@@
 EESchema Schematic File Version 4
+LIBS:ws2812_01sch-cache
 EELAYER 29 0
 EELAYER END
 $Descr A4 11693 8268
 encoding utf-8
-Sheet 1 1
+Sheet 1 7
 Title ""
 Date ""
@@
 $EndDescr
 $Sheet
-S 1550 1500 900  600
+S 1200 5950 900  600
 U 5CD03534
 F0 "esp12" 50
@@
 $EndSheet
 $Sheet
-S 3950 1550 900  600
+S 2750 5950 900  600
+U 5CD03616
+F0 "power_tree" 50
+F1 "power_tree.sch" 50
+$EndSheet
+$Sheet
+S 4550 2050 1550 1050
+U 5CD035B6
+F0 "ws2812_23" 50
+F1 "ws2812_23sch.sch" 50
+F2 "WS2812_IN_ROW1" I L 4550 2150 50
+F3 "WS2812_IN_ROW2" I L 4550 2250 50
+F4 "WS2812_IN_ROW3" I L 4550 2350 50
+F5 "WS2812_IN_ROW4" I L 4550 2450 50
+F6 "WS2812_IN_ROW5" I L 4550 2550 50
+F7 "WS2812_IN_ROW6" I L 4550 2650 50
+F8 "WS2812_IN_ROW7" I L 4550 2750 50
+F9 "WS2812_IN_ROW8" I L 4550 2850 50
+F10 "WS2812_OUT_ROW1" I R 6100 2150 50
+F11 "WS2812_OUT_ROW2" I R 6100 2250 50
+F12 "WS2812_OUT_ROW3" I R 6100 2350 50
+F13 "WS2812_OUT_ROW4" I R 6100 2450 50
+F14 "WS2812_OUT_ROW5" I R 6100 2550 50
+F15 "WS2812_OUT_ROW6" I R 6100 2650 50
+F16 "WS2812_OUT_ROW7" I R 6100 2750 50
+F17 "WS2812_OUT_ROW8" I R 6100 2850 50
+$EndSheet
+$Sheet
+S 6300 2050 1550 1050
+U 5CD08007
+F0 "ws2812_45sch" 50
+F1 "ws2812_45sch.sch" 50
+F2 "WS2812_IN_ROW1" I L 6300 2150 50
+F3 "WS2812_IN_ROW2" I L 6300 2250 50
+F4 "WS2812_IN_ROW3" I L 6300 2350 50
+F5 "WS2812_IN_ROW4" I L 6300 2450 50
+F6 "WS2812_IN_ROW5" I L 6300 2550 50
+F7 "WS2812_IN_ROW6" I L 6300 2650 50
+F8 "WS2812_IN_ROW7" I L 6300 2750 50
+F9 "WS2812_IN_ROW8" I L 6300 2850 50
+F10 "WS2812_OUT_ROW1" I R 7850 2150 50
+F11 "WS2812_OUT_ROW2" I R 7850 2250 50
+F12 "WS2812_OUT_ROW3" I R 7850 2350 50
+F13 "WS2812_OUT_ROW4" I R 7850 2450 50
+F14 "WS2812_OUT_ROW5" I R 7850 2550 50
+F15 "WS2812_OUT_ROW6" I R 7850 2650 50
+F16 "WS2812_OUT_ROW7" I R 7850 2750 50
+F17 "WS2812_OUT_ROW8" I R 7850 2850 50
+$EndSheet
+Wire Wire Line
+	4350 2150 4550 2150
+Wire Wire Line
+	4350 2250 4550 2250
+Wire Wire Line
+	4350 2350 4550 2350
+Wire Wire Line
+	4350 2450 4550 2450
+Wire Wire Line
+	4350 2550 4550 2550
+Wire Wire Line
+	4350 2650 4550 2650
+Wire Wire Line
+	4350 2750 4550 2750
+Wire Wire Line
+	4350 2850 4550 2850
+Wire Wire Line
+	6100 2150 6300 2150
+Wire Wire Line
+	6100 2250 6300 2250
+Wire Wire Line
+	6100 2350 6300 2350
+Wire Wire Line
+	6100 2450 6300 2450
+Wire Wire Line
+	6100 2550 6300 2550
+Wire Wire Line
+	6100 2650 6300 2650
+Wire Wire Line
+	6100 2750 6300 2750
+Wire Wire Line
+	6100 2850 6300 2850
+Wire Wire Line
+	7850 2150 8050 2150
+Wire Wire Line
+	7850 2250 8050 2250
+Wire Wire Line
+	7850 2350 8050 2350
+Wire Wire Line
+	7850 2450 8050 2450
+Wire Wire Line
+	7850 2550 8050 2550
+Wire Wire Line
+	7850 2650 8050 2650
+Wire Wire Line
+	7850 2750 8050 2750
+Wire Wire Line
+	7850 2850 8050 2850
+$Sheet
+S 8050 2050 1550 1050
+U 5CD08019
+F0 "ws2812_67sch" 50
+F1 "ws2812_67sch.sch" 50
+F2 "WS2812_IN_ROW1" I L 8050 2150 50
+F3 "WS2812_IN_ROW2" I L 8050 2250 50
+F4 "WS2812_IN_ROW3" I L 8050 2350 50
+F5 "WS2812_IN_ROW4" I L 8050 2450 50
+F6 "WS2812_IN_ROW5" I L 8050 2550 50
+F7 "WS2812_IN_ROW6" I L 8050 2650 50
+F8 "WS2812_IN_ROW7" I L 8050 2750 50
+F9 "WS2812_IN_ROW8" I L 8050 2850 50
+F10 "WS2812_OUT_ROW1" I R 9600 2150 50
+F11 "WS2812_OUT_ROW2" I R 9600 2250 50
+F12 "WS2812_OUT_ROW3" I R 9600 2350 50
+F13 "WS2812_OUT_ROW4" I R 9600 2450 50
+F14 "WS2812_OUT_ROW5" I R 9600 2550 50
+F15 "WS2812_OUT_ROW6" I R 9600 2650 50
+F16 "WS2812_OUT_ROW7" I R 9600 2750 50
+F17 "WS2812_OUT_ROW8" I R 9600 2850 50
+$EndSheet
+Wire Wire Line
+	9600 2150 9750 2150
+Wire Wire Line
+	9750 2150 9750 2250
+Wire Wire Line
+	9750 2250 9600 2250
+Wire Wire Line
+	9600 2350 9750 2350
+Wire Wire Line
+	9750 2350 9750 2450
+Wire Wire Line
+	9750 2450 9600 2450
+Wire Wire Line
+	9600 2550 9750 2550
+Wire Wire Line
+	9750 2550 9750 2650
+Wire Wire Line
+	9750 2650 9600 2650
+Wire Wire Line
+	9600 2750 9750 2750
+Wire Wire Line
+	9750 2750 9750 2850
+Wire Wire Line
+	9750 2850 9600 2850
+$Sheet
+S 2800 2050 1550 1050
 U 5CD03547
 F0 "ws2812_01" 50
 F1 "ws2812_01sch.sch" 50
-$EndSheet
-$Sheet
-S 5450 1550 900  600
-U 5CD035B6
-F0 "ws2812_23" 50
-F1 "ws2812_23sch.sch" 50
-$EndSheet
-$Sheet
-S 6900 1550 900  600
-U 5CD035EA
-F0 "ws2812_45" 50
-F1 "ws2812_45.sch" 50
-$EndSheet
-$Sheet
-S 8400 1550 900  600
-U 5CD035EC
-F0 "ws2812_67" 50
-F1 "ws2812_67.sch" 50
-$EndSheet
-$Sheet
-S 1550 3200 900  600
-U 5CD03616
-F0 "power_tree" 50
-F1 "power_tree.sch" 50
-$EndSheet
+F2 "WS2812_IN_ROW1" I L 2800 2150 50
+F3 "WS2812_IN_ROW2" I L 2800 2250 50
+F4 "WS2812_IN_ROW3" I L 2800 2350 50
+F5 "WS2812_IN_ROW4" I L 2800 2450 50
+F6 "WS2812_IN_ROW5" I L 2800 2550 50
+F7 "WS2812_IN_ROW6" I L 2800 2650 50
+F8 "WS2812_IN_ROW7" I L 2800 2750 50
+F9 "WS2812_IN_ROW8" I L 2800 2850 50
+F10 "WS2812_OUT_ROW1" I R 4350 2150 50
+F11 "WS2812_OUT_ROW2" I R 4350 2250 50
+F12 "WS2812_OUT_ROW3" I R 4350 2350 50
+F13 "WS2812_OUT_ROW4" I R 4350 2450 50
+F14 "WS2812_OUT_ROW5" I R 4350 2550 50
+F15 "WS2812_OUT_ROW6" I R 4350 2650 50
+F16 "WS2812_OUT_ROW7" I R 4350 2750 50
+F17 "WS2812_OUT_ROW8" I R 4350 2850 50
+$EndSheet
+Wire Wire Line
+	2800 2250 2700 2250
+Wire Wire Line
+	2700 2250 2700 2350
+Wire Wire Line
+	2700 2350 2800 2350
+Wire Wire Line
+	2800 2450 2700 2450
+Wire Wire Line
+	2700 2450 2700 2550
+Wire Wire Line
+	2700 2550 2800 2550
+Wire Wire Line
+	2800 2650 2700 2650
+Wire Wire Line
+	2700 2650 2700 2750
+Wire Wire Line
+	2700 2750 2800 2750
+$Comp
+L Connector_Generic:Conn_01x03 J?
+U 1 1 5CD1A73A
+P 2150 2850
+F 0 "J?" H 2050 3200 50  0000 C CNN
+F 1 "Conn_01x03" H 2050 3100 50  0000 C CNN
+F 2 "" H 2150 2850 50  0001 C CNN
+F 3 "~" H 2150 2850 50  0001 C CNN
+	1    2150 2850
+	-1   0    0    -1
+$EndComp
+$Comp
+L power:VDD #PWR?
+U 1 1 5CD1AFF9
+P 2500 2600
+F 0 "#PWR?" H 2500 2450 50  0001 C CNN
+F 1 "VDD" H 2550 2800 50  0000 C CNN
+F 2 "" H 2500 2600 50  0001 C CNN
+F 3 "" H 2500 2600 50  0001 C CNN
+	1    2500 2600
+	1    0    0    -1
+$EndComp
+Wire Wire Line
+	2500 2600 2500 2750
+Wire Wire Line
+	2500 2750 2350 2750
+Wire Wire Line
+	2350 2850 2800 2850
+$Comp
+L power:GND #PWR?
+U 1 1 5CD1E16F
+P 2500 3150
+F 0 "#PWR?" H 2500 2900 50  0001 C CNN
+F 1 "GND" H 2550 2950 50  0000 C CNN
+F 2 "" H 2500 3150 50  0001 C CNN
+F 3 "" H 2500 3150 50  0001 C CNN
+	1    2500 3150
+	1    0    0    -1
+$EndComp
+Wire Wire Line
+	2500 3150 2500 2950
+Wire Wire Line
+	2500 2950 2350 2950
 $EndSCHEMATC

Commit message: update,
Parts:
- gave numbers to parts that had none: 1
Connections:
- net ws2812_01/WS2812_IN_ROW8: no longer J65.2 (Pin_2)
- net ws2812_01/WS2812_OUT_ROW8: now also J65.2 (Pin_2)
Changed lines of the file:
@@
 EESchema Schematic File Version 4
-LIBS:ws2812_01sch-cache
+LIBS:follower_counter_tryout-cache
 EELAYER 29 0
 EELAYER END
@@
 F1 "ws2812_23sch.sch" 50
 F2 "WS2812_IN_ROW1" I L 4550 2150 50
-F3 "WS2812_IN_ROW2" I L 4550 2250 50
+F3 "WS2812_IN_ROW2" I R 6100 2250 50
 F4 "WS2812_IN_ROW3" I L 4550 2350 50
-F5 "WS2812_IN_ROW4" I L 4550 2450 50
+F5 "WS2812_IN_ROW4" I R 6100 2450 50
 F6 "WS2812_IN_ROW5" I L 4550 2550 50
-F7 "WS2812_IN_ROW6" I L 4550 2650 50
+F7 "WS2812_IN_ROW6" I R 6100 2650 50
 F8 "WS2812_IN_ROW7" I L 4550 2750 50
-F9 "WS2812_IN_ROW8" I L 4550 2850 50
+F9 "WS2812_IN_ROW8" I R 6100 2850 50
 F10 "WS2812_OUT_ROW1" I R 6100 2150 50
-F11 "WS2812_OUT_ROW2" I R 6100 2250 50
+F11 "WS2812_OUT_ROW2" I L 4550 2250 50
 F12 "WS2812_OUT_ROW3" I R 6100 2350 50
-F13 "WS2812_OUT_ROW4" I R 6100 2450 50
+F13 "WS2812_OUT_ROW4" I L 4550 2450 50
 F14 "WS2812_OUT_ROW5" I R 6100 2550 50
-F15 "WS2812_OUT_ROW6" I R 6100 2650 50
+F15 "WS2812_OUT_ROW6" I L 4550 2650 50
 F16 "WS2812_OUT_ROW7" I R 6100 2750 50
-F17 "WS2812_OUT_ROW8" I R 6100 2850 50
+F17 "WS2812_OUT_ROW8" I L 4550 2850 50
 $EndSheet
 $Sheet
@@
 F1 "ws2812_45sch.sch" 50
 F2 "WS2812_IN_ROW1" I L 6300 2150 50
-F3 "WS2812_IN_ROW2" I L 6300 2250 50
+F3 "WS2812_IN_ROW2" I R 7850 2250 50
 F4 "WS2812_IN_ROW3" I L 6300 2350 50
-F5 "WS2812_IN_ROW4" I L 6300 2450 50
+F5 "WS2812_IN_ROW4" I R 7850 2450 50
 F6 "WS2812_IN_ROW5" I L 6300 2550 50
-F7 "WS2812_IN_ROW6" I L 6300 2650 50
+F7 "WS2812_IN_ROW6" I R 7850 2650 50
 F8 "WS2812_IN_ROW7" I L 6300 2750 50
-F9 "WS2812_IN_ROW8" I L 6300 2850 50
+F9 "WS2812_IN_ROW8" I R 7850 2850 50
 F10 "WS2812_OUT_ROW1" I R 7850 2150 50
-F11 "WS2812_OUT_ROW2" I R 7850 2250 50
+F11 "WS2812_OUT_ROW2" I L 6300 2250 50
 F12 "WS2812_OUT_ROW3" I R 7850 2350 50
-F13 "WS2812_OUT_ROW4" I R 7850 2450 50
+F13 "WS2812_OUT_ROW4" I L 6300 2450 50
 F14 "WS2812_OUT_ROW5" I R 7850 2550 50
-F15 "WS2812_OUT_ROW6" I R 7850 2650 50
+F15 "WS2812_OUT_ROW6" I L 6300 2650 50
 F16 "WS2812_OUT_ROW7" I R 7850 2750 50
-F17 "WS2812_OUT_ROW8" I R 7850 2850 50
+F17 "WS2812_OUT_ROW8" I L 6300 2850 50
 $EndSheet
 Wire Wire Line
@@
 F1 "ws2812_67sch.sch" 50
 F2 "WS2812_IN_ROW1" I L 8050 2150 50
-F3 "WS2812_IN_ROW2" I L 8050 2250 50
+F3 "WS2812_IN_ROW2" I R 9600 2250 50
 F4 "WS2812_IN_ROW3" I L 8050 2350 50
-F5 "WS2812_IN_ROW4" I L 8050 2450 50
+F5 "WS2812_IN_ROW4" I R 9600 2450 50
 F6 "WS2812_IN_ROW5" I L 8050 2550 50
-F7 "WS2812_IN_ROW6" I L 8050 2650 50
+F7 "WS2812_IN_ROW6" I R 9600 2650 50
 F8 "WS2812_IN_ROW7" I L 8050 2750 50
-F9 "WS2812_IN_ROW8" I L 8050 2850 50
+F9 "WS2812_IN_ROW8" I R 9600 2850 50
 F10 "WS2812_OUT_ROW1" I R 9600 2150 50
-F11 "WS2812_OUT_ROW2" I R 9600 2250 50
+F11 "WS2812_OUT_ROW2" I L 8050 2250 50
 F12 "WS2812_OUT_ROW3" I R 9600 2350 50
-F13 "WS2812_OUT_ROW4" I R 9600 2450 50
+F13 "WS2812_OUT_ROW4" I L 8050 2450 50
 F14 "WS2812_OUT_ROW5" I R 9600 2550 50
-F15 "WS2812_OUT_ROW6" I R 9600 2650 50
+F15 "WS2812_OUT_ROW6" I L 8050 2650 50
 F16 "WS2812_OUT_ROW7" I R 9600 2750 50
-F17 "WS2812_OUT_ROW8" I R 9600 2850 50
+F17 "WS2812_OUT_ROW8" I L 8050 2850 50
 $EndSheet
 Wire Wire Line
@@
 F1 "ws2812_01sch.sch" 50
 F2 "WS2812_IN_ROW1" I L 2800 2150 50
-F3 "WS2812_IN_ROW2" I L 2800 2250 50
+F3 "WS2812_IN_ROW2" I R 4350 2250 50
 F4 "WS2812_IN_ROW3" I L 2800 2350 50
-F5 "WS2812_IN_ROW4" I L 2800 2450 50
+F5 "WS2812_IN_ROW4" I R 4350 2450 50
 F6 "WS2812_IN_ROW5" I L 2800 2550 50
-F7 "WS2812_IN_ROW6" I L 2800 2650 50
+F7 "WS2812_IN_ROW6" I R 4350 2650 50
 F8 "WS2812_IN_ROW7" I L 2800 2750 50
-F9 "WS2812_IN_ROW8" I L 2800 2850 50
+F9 "WS2812_IN_ROW8" I R 4350 2850 50
 F10 "WS2812_OUT_ROW1" I R 4350 2150 50
-F11 "WS2812_OUT_ROW2" I R 4350 2250 50
+F11 "WS2812_OUT_ROW2" I L 2800 2250 50
 F12 "WS2812_OUT_ROW3" I R 4350 2350 50
-F13 "WS2812_OUT_ROW4" I R 4350 2450 50
+F13 "WS2812_OUT_ROW4" I L 2800 2450 50
 F14 "WS2812_OUT_ROW5" I R 4350 2550 50
-F15 "WS2812_OUT_ROW6" I R 4350 2650 50
+F15 "WS2812_OUT_ROW6" I L 2800 2650 50
 F16 "WS2812_OUT_ROW7" I R 4350 2750 50
-F17 "WS2812_OUT_ROW8" I R 4350 2850 50
+F17 "WS2812_OUT_ROW8" I L 2800 2850 50
 $EndSheet
 Wire Wire Line
@@
 	2700 2750 2800 2750
 $Comp
-L Connector_Generic:Conn_01x03 J?
+L Connector_Generic:Conn_01x03 J65
 U 1 1 5CD1A73A
 P 2150 2850
-F 0 "J?" H 2050 3200 50  0000 C CNN
+F 0 "J65" H 2050 3200 50  0000 C CNN
 F 1 "Conn_01x03" H 2050 3100 50  0000 C CNN
 F 2 "" H 2150 2850 50  0001 C CNN
@@
 $EndComp
 $Comp
-L power:VDD #PWR?
+L power:VDD #PWR0129
 U 1 1 5CD1AFF9
 P 2500 2600
-F 0 "#PWR?" H 2500 2450 50  0001 C CNN
+F 0 "#PWR0129" H 2500 2450 50  0001 C CNN
 F 1 "VDD" H 2550 2800 50  0000 C CNN
 F 2 "" H 2500 2600 50  0001 C CNN
@@
 	2350 2850 2800 2850
 $Comp
-L power:GND #PWR?
+L power:GND #PWR0130
 U 1 1 5CD1E16F
 P 2500 3150
-F 0 "#PWR?" H 2500 2900 50  0001 C CNN
+F 0 "#PWR0130" H 2500 2900 50  0001 C CNN
 F 1 "GND" H 2550 2950 50  0000 C CNN
 F 2 "" H 2500 3150 50  0001 C CNN

Commit message: update,
Other:
- moved on the sheet: J65
