File: hardware/follower_counter_tryout.sch (KiCad schematic (older format))
At the start: 1 part, among them J65 Conn_01x03

Commit message: update WS2812\,
Parts:
- J65: value Conn_01x03 -> WS2812_OUT
Changed lines of the file:
@@
 $Descr A4 11693 8268
 encoding utf-8
-Sheet 1 12
+Sheet 1 11
 Title ""
 Date ""
@@
 P 3300 3750
 F 0 "J65" H 3200 4100 50  0000 C CNN
-F 1 "Conn_01x03" H 3200 4000 50  0000 C CNN
+F 1 "WS2812_OUT" H 3200 4000 50  0000 C CNN
 F 2 "" H 3300 3750 50  0001 C CNN
 F 3 "~" H 3300 3750 50  0001 C CNN
