File: hardware/ws2812_01sch.sch (KiCad schematic (older format))
At the start: 64 parts

Commit message: update,
Parts:
- removed D? (x32): WS2812B, footprint-lib:LED_WS2812B_PLCC4_5.0x5.0mm_P3.2mm, symbol LED:WS2812B
- added D11, D12, D15, D16, D17, D21, D22, D25, D26, D28, D29, D30, D33, D34, D36, D39, D4, D40, D41, D42, D43, D44, D49, D5, D55, D57, D60, D61, D63, D64, D7, D8: WS2812B, footprint-lib:LED_WS2812B_PLCC4_5.0x5.0mm_P3.2mm, symbol LED:WS2812B
- gave numbers to parts that had none: 32
Connections:
- net GND: now also D11.3 (VSS), D12.3 (VSS), D15.3 (VSS), D16.3 (VSS), D17.3 (VSS), D21.3 (VSS), D22.3 (VSS), D25.3 (VSS), D26.3 (VSS), D28.3 (VSS), D29.3 (VSS), D30.3 (VSS), D33.3 (VSS), D34.3 (VSS), D36.3 (VSS), D39.3 (VSS), D4.3 (VSS), D40.3 (VSS), D41.3 (VSS), D42.3 (VSS), D43.3 (VSS), D44.3 (VSS), D49.3 (VSS), D5.3 (VSS), D55.3 (VSS), D57.3 (VSS), D60.3 (VSS), D61.3 (VSS), D63.3 (VSS), D64.3 (VSS), D7.3 (VSS), D8.3 (VSS)
- net VDD: now also D11.1 (VDD), D12.1 (VDD), D15.1 (VDD), D16.1 (VDD), D17.1 (VDD), D21.1 (VDD), D22.1 (VDD), D25.1 (VDD), D26.1 (VDD), D28.1 (VDD), D29.1 (VDD), D30.1 (VDD), D33.1 (VDD), D34.1 (VDD), D36.1 (VDD), D39.1 (VDD), D4.1 (VDD), D40.1 (VDD), D41.1 (VDD), D42.1 (VDD), D43.1 (VDD), D44.1 (VDD), D49.1 (VDD), D5.1 (VDD), D55.1 (VDD), D57.1 (VDD), D60.1 (VDD), D61.1 (VDD), D63.1 (VDD), D64.1 (VDD), D7.1 (VDD), D8.1 (VDD)
- net WS2812_IN_ROW3: now also D17.4 (DIN)
- net WS2812_IN_ROW4: now also D25.4 (DIN)
- net WS2812_IN_ROW5: now also D33.4 (DIN)
- net WS2812_IN_ROW6: now also D41.4 (DIN)
- net WS2812_IN_ROW7: now also D49.4 (DIN)
- net WS2812_IN_ROW8: now also D57.4 (DIN)
- net WS2812_OUT_ROW1: now also D8.2 (DOUT)
- net WS2812_OUT_ROW2: now also D16.2 (DOUT)
- net WS2812_OUT_ROW5: now also D40.2 (DOUT)
- net WS2812_OUT_ROW8: now also D64.2 (DOUT)
- net at D6.2 (DOUT): now also D7.4 (DIN)
- net at D6.4 (DIN): now also D5.2 (DOUT)
- net at D10.2 (DOUT): now also D11.4 (DIN)
- net at D20.2 (DOUT): now also D21.4 (DIN)
- net at D23.4 (DIN): now also D22.2 (DOUT)
- net at D31.4 (DIN): now also D30.2 (DOUT)
- net at D50.4 (DIN): now also D49.2 (DOUT)
- net at D54.2 (DOUT): now also D55.4 (DIN)
- net at D58.4 (DIN): now also D57.2 (DOUT)
- net at D59.2 (DOUT): now also D60.4 (DIN)
- net at D62.2 (DOUT): now also D63.4 (DIN)
- net at D35.4 (DIN): now also D34.2 (DOUT)
- net at D35.2 (DOUT): now also D36.4 (DIN)
- net at D45.4 (DIN): now also D44.2 (DOUT)
- net at D3.2 (DOUT): now also D4.4 (DIN)
- net at D13.4 (DIN): now also D12.2 (DOUT)
- net at D18.4 (DIN): now also D17.2 (DOUT)
- net at D37.4 (DIN): now also D36.2 (DOUT)
- net at D38.2 (DOUT): now also D39.4 (DIN)
- net at D56.4 (DIN): now also D55.2 (DOUT)
- net at D62.4 (DIN): now also D61.2 (DOUT)
- net at D14.2 (DOUT): now also D15.4 (DIN)
- net at D27.4 (DIN): now also D26.2 (DOUT)
- net at D27.2 (DOUT): now also D28.4 (DIN)
- new net: D11.2 (DOUT), D12.4 (DIN)
- new net: D29.2 (DOUT), D30.4 (DIN)
- new net: D28.2 (DOUT), D29.4 (DIN)
- new net: D42.2 (DOUT), D43.4 (DIN)
- new net: D41.2 (DOUT), D42.4 (DIN)
- new net: D63.2 (DOUT), D64.4 (DIN)
- new net: D33.2 (DOUT), D34.4 (DIN)
- new net: D43.2 (DOUT), D44.4 (DIN)
- new net: D4.2 (DOUT), D5.4 (DIN)
- new net: D7.2 (DOUT), D8.4 (DIN)
- new net: D21.2 (DOUT), D22.4 (DIN)
- new net: D39.2 (DOUT), D40.4 (DIN)
- new net: D60.2 (DOUT), D61.4 (DIN)
- new net: D15.2 (DOUT), D16.4 (DIN)
- new net: D25.2 (DOUT), D26.4 (DIN)
