File: hardware/ws2812_45sch.sch (KiCad schematic (older format))
At the start: 64 parts

Commit message: update,
Parts:
- removed D? (x32): WS2812B, footprint-lib:LED_WS2812B_PLCC4_5.0x5.0mm_P3.2mm, symbol LED:WS2812B
- added D129, D130, D131, D134, D137, D138, D141, D142, D146, D147, D148, D151, D152, D155, D159, D160, D163, D165, D166, D173, D174, D175, D176, D178, D179, D180, D181, D182, D184, D186, D187, D190: WS2812B, footprint-lib:LED_WS2812B_PLCC4_5.0x5.0mm_P3.2mm, symbol LED:WS2812B
- gave numbers to parts that had none: 32
Connections:
- net GND: now also D129.3 (VSS), D130.3 (VSS), D131.3 (VSS), D134.3 (VSS), D137.3 (VSS), D138.3 (VSS), D141.3 (VSS), D142.3 (VSS), D146.3 (VSS), D147.3 (VSS), D148.3 (VSS), D151.3 (VSS), D152.3 (VSS), D155.3 (VSS), D159.3 (VSS), D160.3 (VSS), D163.3 (VSS), D165.3 (VSS), D166.3 (VSS), D173.3 (VSS), D174.3 (VSS), D175.3 (VSS), D176.3 (VSS), D178.3 (VSS), D179.3 (VSS), D180.3 (VSS), D181.3 (VSS), D182.3 (VSS), D184.3 (VSS), D186.3 (VSS), D187.3 (VSS), D190.3 (VSS)
- net VDD: now also D129.1 (VDD), D130.1 (VDD), D131.1 (VDD), D134.1 (VDD), D137.1 (VDD), D138.1 (VDD), D141.1 (VDD), D142.1 (VDD), D146.1 (VDD), D147.1 (VDD), D148.1 (VDD), D151.1 (VDD), D152.1 (VDD), D155.1 (VDD), D159.1 (VDD), D160.1 (VDD), D163.1 (VDD), D165.1 (VDD), D166.1 (VDD), D173.1 (VDD), D174.1 (VDD), D175.1 (VDD), D176.1 (VDD), D178.1 (VDD), D179.1 (VDD), D180.1 (VDD), D181.1 (VDD), D182.1 (VDD), D184.1 (VDD), D186.1 (VDD), D187.1 (VDD), D190.1 (VDD)
- net WS2812_IN_ROW1: now also D129.4 (DIN)
- net WS2812_IN_ROW2: now also D137.4 (DIN)
- net WS2812_OUT_ROW3: now also D152.2 (DOUT)
- net WS2812_OUT_ROW4: now also D160.2 (DOUT)
- net WS2812_OUT_ROW6: now also D176.2 (DOUT)
- net WS2812_OUT_ROW7: now also D184.2 (DOUT)
- net at D135.4 (DIN): now also D134.2 (DOUT)
- net at D133.2 (DOUT): now also D134.4 (DIN)
- net at D139.4 (DIN): now also D138.2 (DOUT)
- net at D149.4 (DIN): now also D148.2 (DOUT)
- net at D150.2 (DOUT): now also D151.4 (DIN)
- net at D158.2 (DOUT): now also D159.4 (DIN)
- net at D177.2 (DOUT): now also D178.4 (DIN)
- net at D183.4 (DIN): now also D182.2 (DOUT)
- net at D185.2 (DOUT): now also D186.4 (DIN)
- net at D188.4 (DIN): now also D187.2 (DOUT)
- net at D191.4 (DIN): now also D190.2 (DOUT)
- net at D162.2 (DOUT): now also D163.4 (DIN)
- net at D164.4 (DIN): now also D163.2 (DOUT)
- net at D172.2 (DOUT): now also D173.4 (DIN)
- net at D132.4 (DIN): now also D131.2 (DOUT)
- net at D140.2 (DOUT): now also D141.4 (DIN)
- net at D145.2 (DOUT): now also D146.4 (DIN)
- net at D164.2 (DOUT): now also D165.4 (DIN)
- net at D167.4 (DIN): now also D166.2 (DOUT)
- net at D183.2 (DOUT): now also D184.4 (DIN)
- net at D189.2 (DOUT): now also D190.4 (DIN)
- net at D143.4 (DIN): now also D142.2 (DOUT)
- net at D154.2 (DOUT): now also D155.4 (DIN)
- net at D156.4 (DIN): now also D155.2 (DOUT)
- new net: D147.2 (DOUT), D148.4 (DIN)
- new net: D146.2 (DOUT), D147.4 (DIN)
- new net: D151.2 (DOUT), D152.4 (DIN)
- new net: D159.2 (DOUT), D160.4 (DIN)
- new net: D175.2 (DOUT), D176.4 (DIN)
- new net: D174.2 (DOUT), D175.4 (DIN)
- new net: D180.2 (DOUT), D181.4 (DIN)
- new net: D179.2 (DOUT), D180.4 (DIN)
- new net: D181.2 (DOUT), D182.4 (DIN)
- new net: D186.2 (DOUT), D187.4 (DIN)
- new net: D173.2 (DOUT), D174.4 (DIN)
- new net: D178.2 (DOUT), D179.4 (DIN)
- new net: D130.2 (DOUT), D131.4 (DIN)
- new net: D129.2 (DOUT), D130.4 (DIN)
- new net: D137.2 (DOUT), D138.4 (DIN)
- new net: D141.2 (DOUT), D142.4 (DIN)
- new net: D165.2 (DOUT), D166.4 (DIN)
