File: hardware/ws2812_67sch.sch (KiCad schematic (older format))
At the start: 64 parts

Commit message: update,
Parts:
- removed D? (x24): WS2812B, footprint-lib:LED_WS2812B_PLCC4_5.0x5.0mm_P3.2mm, symbol LED:WS2812B
- added D194, D195, D196, D198, D199, D202, D204, D205, D216, D223, D224, D226, D227, D229, D230, D232, D234, D237, D238, D241, D242, D243, D250, D254: WS2812B, footprint-lib:LED_WS2812B_PLCC4_5.0x5.0mm_P3.2mm, symbol LED:WS2812B
- gave numbers to parts that had none: 40
Connections:
- net GND: now also D194.3 (VSS), D195.3 (VSS), D196.3 (VSS), D198.3 (VSS), D199.3 (VSS), D202.3 (VSS), D204.3 (VSS), D205.3 (VSS), D216.3 (VSS), D223.3 (VSS), D224.3 (VSS), D226.3 (VSS), D227.3 (VSS), D229.3 (VSS), D230.3 (VSS), D232.3 (VSS), D234.3 (VSS), D237.3 (VSS), D238.3 (VSS), D241.3 (VSS), D242.3 (VSS), D243.3 (VSS), D250.3 (VSS), D254.3 (VSS)
- net VDD: now also D194.1 (VDD), D195.1 (VDD), D196.1 (VDD), D198.1 (VDD), D199.1 (VDD), D202.1 (VDD), D204.1 (VDD), D205.1 (VDD), D216.1 (VDD), D223.1 (VDD), D224.1 (VDD), D226.1 (VDD), D227.1 (VDD), D229.1 (VDD), D230.1 (VDD), D232.1 (VDD), D234.1 (VDD), D237.1 (VDD), D238.1 (VDD), D241.1 (VDD), D242.1 (VDD), D243.1 (VDD), D250.1 (VDD), D254.1 (VDD)
- net WS2812_IN_ROW7: now also D241.4 (DIN)
- net WS2812_OUT_ROW3: now also D216.2 (DOUT)
- net WS2812_OUT_ROW4: now also D224.2 (DOUT)
- net WS2812_OUT_ROW5: now also D232.2 (DOUT)
- net at D193.2 (DOUT): now also D194.4 (DIN)
- net at D197.2 (DOUT): now also D198.4 (DIN)
- net at D197.4 (DIN): now also D196.2 (DOUT)
- net at D200.4 (DIN): now also D199.2 (DOUT)
- net at D203.2 (DOUT): now also D204.4 (DIN)
- net at D215.2 (DOUT): now also D216.4 (DIN)
- net at D228.2 (DOUT): now also D229.4 (DIN)
- net at D228.4 (DIN): now also D227.2 (DOUT)
- net at D231.2 (DOUT): now also D232.4 (DIN)
- net at D231.4 (DIN): now also D230.2 (DOUT)
- net at D253.2 (DOUT): now also D254.4 (DIN)
- net at D255.4 (DIN): now also D254.2 (DOUT)
- net at D201.2 (DOUT): now also D202.4 (DIN)
- net at D203.4 (DIN): now also D202.2 (DOUT)
- net at D206.4 (DIN): now also D205.2 (DOUT)
- net at D233.2 (DOUT): now also D234.4 (DIN)
- net at D239.4 (DIN): now also D238.2 (DOUT)
- net at D222.2 (DOUT): now also D223.4 (DIN)
- net at D235.4 (DIN): now also D234.2 (DOUT)
- net at D244.4 (DIN): now also D243.2 (DOUT)
- net at D249.2 (DOUT): now also D250.4 (DIN)
- net at D251.4 (DIN): now also D250.2 (DOUT)
- net at D225.2 (DOUT): now also D226.4 (DIN)
- net at D236.2 (DOUT): now also D237.4 (DIN)
- new net: D194.2 (DOUT), D195.4 (DIN)
- new net: D195.2 (DOUT), D196.4 (DIN)
- new net: D198.2 (DOUT), D199.4 (DIN)
- new net: D204.2 (DOUT), D205.4 (DIN)
- new net: D242.2 (DOUT), D243.4 (DIN)
- new net: D241.2 (DOUT), D242.4 (DIN)
- new net: D229.2 (DOUT), D230.4 (DIN)
- new net: D237.2 (DOUT), D238.4 (DIN)
- new net: D223.2 (DOUT), D224.4 (DIN)
- new net: D226.2 (DOUT), D227.4 (DIN)
