File: hardware/esp12_core.sch (KiCad schematic (older format))
At the start: 8 parts

Commit message: update ESP12 core,
Connections:
- net +3V3: now also U?.8 (VDD)
- net GND: now also U?.15 (GND)
Changed lines of the file:
@@
 $Descr A4 11693 8268
 encoding utf-8
-Sheet 3 11
+Sheet 3 12
 Title ""
 Date ""
@@
 F1 "ESP12_button.sch" 50
 $EndSheet
+$Sheet
+S 7600 2750 950  700
+U 5CD78B17
+F0 "ADC" 50
+F1 "ADC.sch" 50
+$EndSheet
+$Comp
+L power:+3V3 #PWR?
+U 1 1 5CD7B601
+P 3600 3900
+F 0 "#PWR?" H 3600 3750 50  0001 C CNN
+F 1 "+3V3" H 3650 4100 50  0000 C CNN
+F 2 "" H 3600 3900 50  0001 C CNN
+F 3 "" H 3600 3900 50  0001 C CNN
+	1    3600 3900
+	1    0    0    -1
+$EndComp
+$Comp
+L power:GND #PWR?
+U 1 1 5CD7BA45
+P 3600 6200
+F 0 "#PWR?" H 3600 5950 50  0001 C CNN
+F 1 "GND" H 3650 6000 50  0000 C CNN
+F 2 "" H 3600 6200 50  0001 C CNN
+F 3 "" H 3600 6200 50  0001 C CNN
+	1    3600 6200
+	1    0    0    -1
+$EndComp
+Wire Wire Line
+	3600 6050 3600 6200
+Wire Wire Line
+	3600 3900 3600 4100
 $EndSCHEMATC
